Commit message: Complete Gazebo setup

File: src/mecanum_robot/urdf/mecanum_robot.urdf.xacro (robot description, xacro)
@@ -40,14 +40,13 @@
       <origin xyz="0 0 ${0.0251 + (0.1201 - 0.0251) / 2}" rpy="0 0 0" />
       <geometry>
-        <box size="${chassis_length} ${chassis_width} ${chassis_height}" />
+        <box size="${chassis_width} ${chassis_length} ${chassis_height}" />
       </geometry>
     </collision>
     <inertial>
       <mass value="${chassis_mass}" />
-      <origin xyz="0 0 ${chassis_height / 2}" rpy="0 0 0" />
-      <!-- Box inertia approximation — replace with SolidWorks values if you have them -->
+      <origin xyz="0 0 ${0.0251 + (0.1201 - 0.0251) / 2}" rpy="0 0 0" />
       <inertia
-        ixx="0.0079" ixy="0" ixz="0"
-        iyy="0.0064" iyz="0.0003" izz="0.0065" />
+        ixx="0.0064" ixy="0" ixz="0"
+        iyy="0.0079" iyz="0" izz="0.0065" />
     </inertial>
   </link>
@@ -69,10 +68,4 @@
         </material>
       </visual>
-      <collision>
-        <origin xyz="0 0 0" rpy="${pi/2} 0 0" />
-        <geometry>
-          <cylinder radius="${wheel_radius}" length="${wheel_width}" />
-        </geometry>
-      </collision>
       <inertial>
         <mass value="${wheel_mass}" />
@@ -114,8 +107,8 @@
           <scan>
             <horizontal>
-              <samples>1</samples>
+              <samples>5</samples>
               <resolution>1</resolution>
-              <min_angle>0</min_angle>
-              <max_angle>0</max_angle>
+              <min_angle>-0.22</min_angle>
+              <max_angle>0.22</max_angle>
             </horizontal>
           </scan>
@@ -165,27 +158,33 @@
     </plugin>
   </gazebo>
-  <!-- Gazebo material colors (Gazebo ignores URDF materials, needs its own) -->
-  <gazebo reference="chassis_link">
-    <material>Gazebo/Grey</material>
-  </gazebo>
   <gazebo reference="front_left_wheel_link">
     <material>Gazebo/DarkGrey</material>
-    <mu1>1.0</mu1>
-    <mu2>1.0</mu2>
+    <mu1>0.001</mu1>
+    <mu2>0.001</mu2>
+    <gravity>false</gravity>
   </gazebo>
   <gazebo reference="front_right_wheel_link">
     <material>Gazebo/DarkGrey</material>
-    <mu1>1.0</mu1>
-    <mu2>1.0</mu2>
+    <mu1>0.001</mu1>
+    <mu2>0.001</mu2>
+    <gravity>false</gravity>
   </gazebo>
-  <gazebo reference="rear_left_wheel_link">
+  <gazebo reference="back_left_wheel_link">
     <material>Gazebo/DarkGrey</material>
-    <mu1>1.0</mu1>
-    <mu2>1.0</mu2>
+    <mu1>0.001</mu1>
+    <mu2>0.001</mu2>
+    <gravity>false</gravity>
   </gazebo>
-  <gazebo reference="rear_right_wheel_link">
+  <gazebo reference="back_right_wheel_link">
     <material>Gazebo/DarkGrey</material>
-    <mu1>1.0</mu1>
-    <mu2>1.0</mu2>
+    <mu1>0.001</mu1>
+    <mu2>0.001</mu2>
+    <gravity>false</gravity>
+  </gazebo>
+  <gazebo reference="chassis_link">
+    <material>Gazebo/Grey</material>
+    <mu1>0.001</mu1>
+    <mu2>0.001</mu2>
+    <gravity>false</gravity>
   </gazebo>
 </robot>
